Commit message: debugged urdf with realsense, debugged map/path-related launch files

File: urdf/rallycar.urdf (robot description, URDF)
Before this commit: robot rallycar, 4 links, 3 joints
Links:
- removed link rs_camera
- added link rs_camera_link
Joints:
- joint base_to_real_sense: child rs_camera -> rs_camera_link
